File: Dingo-75.kicad_pcb (KiCad board)
At the start: 2 copper layers, 344.5 x 123.8 mm, 178 parts, among them SW1 SW_Push, U1 AT90USB1286-AU, Y1 16MHz

Commit message: Completed routing
Parts:
- C4: moved to F.Cu
- moved C5 34.4 mm to (76.5, -200.8), turned to 180 degrees
- moved C2 27.1 mm to (71.1, -192.8), turned to 180 degrees
- moved C3 26.6 mm to (61.2, -188.1), turned to 270 degrees
- moved C4 25.0 mm to (60.1, -178.5)
- moved R1 8.31 mm to (70.2, -169.5), turned to 270 degrees
- moved R4 4.18 mm to (83.8, -191.5)
- moved C1 3.89 mm to (74.6, -203.7), turned to 0 degrees
- moved R3 0.96 mm to (67.6, -201.6)
- moved R2 0.61 mm to (69.7, -201.6)
Connections:
- MX'1 pad 1: Col9 -> Col11
- MX,1 pad 1: Col7 -> Col9
- MX-1 pad 1: Col9 -> Col11
- MX-Alt1 pad 1: Col1 -> Col2
- MX-Alt2 pad 1: Col7 -> Col8
- MX-Back1 pad 1: Col11 -> Col13
- MX-Ctrl2 pad 1: Net-(MX-Ctrl2-Pad1) -> Col10
- MX-Delete1 pad 1: Col13 -> Col14
- MX-Down1 pad 1: Col11 -> Col13
- MX-End1 pad 1: Col13 -> Col14
- MX-Enter1 pad 1: Col11 -> Col13
- MX-Fn1 pad 1: Col8 -> Col9
- MX-Home1 pad 1: Col13 -> Col14
- MX-Insert1 pad 1: Col13 -> Col14
- MX-Left1 pad 1: Col9 -> Col11
- MX-Right1 pad 1: Col13 -> Col14
- MX-Shift2 pad 1: Col11 -> Col13
- MX-Space1 pad 1: Col4 -> Col6
- MX-Up1 pad 1: Col13 -> Col14
- MX-Win1 pad 1: Net-(MX-Win1-Pad1) -> Col1
- MX.1 pad 1: Col8 -> Col10
- MX/1 pad 1: Net-(MX-Ctrl2-Pad1) -> Col11
- MX0 pad 1: Net-(MX-Ctrl2-Pad1) -> Col10
- MX1 pad 1: Net-(MX-Win1-Pad1) -> Col1
- MX2 pad 1: Col1 -> Col2
- MX3 pad 1: Col2 -> Col3
- MX4 pad 1: Col3 -> Col4
- MX5 pad 1: Col4 -> Col5
- MX6 pad 1: Col5 -> Col6
- MX7 pad 1: Col6 -> Col7
- MX8 pad 1: Col7 -> Col8
- MX9 pad 1: Col8 -> Col9
- MX;1 pad 1: Net-(MX-Ctrl2-Pad1) -> Col10
- MX=1 pad 1: Col10 -> Col12
- MXA1 pad 1: Net-(MX-Win1-Pad1) -> Col1
- MXB1 pad 1: Col4 -> Col6
- MXC1 pad 1: Col2 -> Col4
- MXD1 pad 1: Col2 -> Col3
- MXE1 pad 1: Col2 -> Col3
- MXF-1 pad 1: Col3 -> Col4
- MXF1 pad 1: Col1 -> Col2
- MXF10 pad 1: Col10 -> Col11
- MXF11 pad 1: Col11 -> Col12
- MXF12 pad 1: Col12 -> Col13
- MXF2 pad 1: Col2 -> Col3
- MXF3 pad 1: Col3 -> Col4
- MXF4 pad 1: Col4 -> Col5
- MXF5 pad 1: Col5 -> Col6
- MXF6 pad 1: Col6 -> Col7
- MXF7 pad 1: Col7 -> Col8
- MXF8 pad 1: Col8 -> Col9
- MXF9 pad 1: Col9 -> Col10
- MXG1 pad 1: Col4 -> Col5
- MXH1 pad 1: Col5 -> Col6
- MXI1 pad 1: Col7 -> Col8
- MXJ1 pad 1: Col6 -> Col7
- MXK1 pad 1: Col7 -> Col8
- MXL1 pad 1: Col8 -> Col9
- MXM1 pad 1: Col6 -> Col8
- MXN1 pad 1: Col5 -> Col7
- MXO1 pad 1: Col8 -> Col9
- MXP1 pad 1: Net-(MX-Ctrl2-Pad1) -> Col10
- MXQ1 pad 1: Net-(MX-Win1-Pad1) -> Col1
- MXR1 pad 1: Col3 -> Col4
- MXS1 pad 1: Col1 -> Col2
- MXT1 pad 1: Col4 -> Col5
- MXU1 pad 1: Col6 -> Col7
- MXV1 pad 1: Col3 -> Col5
- MXW1 pad 1: Col1 -> Col2
- MXX1 pad 1: Net-(MXX1-Pad1) -> Col3
- MXY1 pad 1: Col5 -> Col6
- MXZ1 pad 1: Col1 -> Col2
- MX[1 pad 1: Col9 -> Col11
- MX\1 pad 1: Col11 -> Col13
- MX]1 pad 1: Col10 -> Col12
- U1 pad 38: Net-(U1-Pad38) -> Col0
- U1 pad 39: Net-(U1-Pad39) -> Col1
- U1 pad 40: Net-(U1-Pad40) -> Col2
- U1 pad 41: Net-(U1-Pad41) -> Col3
- U1 pad 42: Net-(U1-Pad42) -> Col4
- U1 pad 44: Net-(U1-Pad44) -> Col5
- U1 pad 45: Net-(U1-Pad45) -> Col6
- U1 pad 46: Net-(U1-Pad46) -> Col7
- U1 pad 47: Net-(U1-Pad47) -> Col8
- U1 pad 48: Net-(U1-Pad48) -> Col9
- U1 pad 49: Net-(U1-Pad49) -> Col10
- U1 pad 50: Net-(U1-Pad50) -> Col11
- U1 pad 51: Net-(U1-Pad51) -> Col12
- U1 pad 54: Row5 -> Col13
- U1 pad 55: Col0 -> Col14
Routing:
- net Col2: track 87.2 -> 497.7 mm, vias 0 -> 1
- net Net-(MX-Win1-Pad1): track 397.0 -> 0.00 mm
- net Col3: track 89.0 -> 470.4 mm, vias 0 -> 1
- net Col5: track 90.9 -> 438.1 mm, vias 0 -> 1
- net Col4: track 110.9 -> 453.6 mm, vias 0 -> 1
- net Col6: track 94.8 -> 417.3 mm, vias 0 -> 1
- net Col10: track 46.8 -> 338.1 mm, vias 0 -> 1
- net Col12: track 0.00 -> 282.5 mm, vias 0 -> 1
- net Col7: track 119.8 -> 395.3 mm, vias 0 -> 1
- net Col8: track 125.4 -> 373.3 mm, vias 0 -> 1
- net Col14: track 0.00 -> 228.8 mm, vias 0 -> 1
- net Col9: track 131.7 -> 353.2 mm, vias 0 -> 1
- net Col11: track 138.4 -> 316.7 mm, vias 0 -> 1
- net Col13: track 114.0 -> 270.2 mm, vias 0 -> 1
- net Net-(MX-Ctrl2-Pad1): track 105.8 -> 0.00 mm
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Other:
- board size 344.5 x 123.8 mm -> 344.5 x 124.5 mm

Commit message: FINISHED V1
Routing:
- net Col3: track 470.4 -> 459.0 mm
- net Col2: track 497.7 -> 490.7 mm
- net Col1: track 484.9 -> 479.7 mm
- net Col0: track 529.0 -> 526.3 mm
- net Col7: track 395.3 -> 393.8 mm
- net Row0: track 323.4 -> 324.2 mm
- net Col5: track 438.1 -> 437.4 mm
- added copper zone on F.Cu, net GND

Commit message: Added finishing touches, including Silkscreening using Images
Parts:
- added G***: LOGO, Dingo-75:David Logo, F.Cu at (-154.4, -105.2)
- added G***: LOGO, Dingo-75:Dingo-Logo, F.Cu at (-91.6, -105.9)
- added G***: LOGO, Dingo-75:Dingo-Path, B.Cu at (63.8, -153.9)
- added H1: MountingHole, MountingHole:MountingHole_2mm, F.Cu at (-214.1, -124.4)
- added H2: MountingHole, MountingHole:MountingHole_2mm, F.Cu at (-16.4, -127.1)
- added H3: MountingHole, MountingHole:MountingHole_2mm, F.Cu at (-228.6, -193.0)
- added H4: MountingHole, MountingHole:MountingHole_2mm, F.Cu at (30.8, -193.0)
Routing:
- net Row0: track 324.2 -> 323.4 mm
